Commit message: Removed link7 and joint7

File: src/xarm_ros/xarm_description/urdf/lite6/lite6.gazebo.xacro (robot description, xacro)
@@ -23,4 +23,7 @@
       <selfCollide>true</selfCollide>
     </gazebo>
+    <gazebo reference="${prefix}link7">
+      <selfCollide>true</selfCollide>
+    </gazebo>
   </xacro:macro>
 </robot>

File: src/xarm_ros/xarm_description/urdf/lite6/lite6.urdf.xacro (robot description, xacro)
@@ -210,31 +210,4 @@
     </joint>
     <!--############ Attach openmanipulatorX link here-->
-    <link name="${prefix}link7">
-      <xacro:common_link_inertial
-        link_inertial_params="${inertial_params['link7']}"
-        origin_rpy="0 0 0"/>
-      <xacro:common_link_visual
-        mesh_filename="lite6/visual/link7"
-        origin_xyz="0 0 0"
-        origin_rpy="0 0 0"
-        material_name="${prefix}Silver" />
-      <xacro:common_link_collision
-        mesh_filename="lite6/collision/link7"
-        origin_xyz="0 0 0"
-        origin_rpy="0 0 0" />
-    </link>
-    <joint name="${prefix}joint7" type="fixed">
-      <!-- <origin xyz="0 0.0625 0" rpy="-1.5708 0 0" /> -->
-      <xacro:common_joint_origin joint_kinematic_params="${kinematics_params['joint7']}" />
-      <parent link="${prefix}link6" />
-      <child link="${prefix}link7" />
-      <axis xyz="0 0 1" />
-      <limit
-        lower="${joint7_lower_limit}"
-        upper="${joint7_upper_limit}"
-        effort="20.0"
-        velocity="3.14"/>
-      <dynamics damping="1.0" friction="1.0"/>
-    </joint>
     <!-- <link name="${prefix}link_eef" />
     <joint name="${prefix}joint_eef" type="fixed">
