Commit message: Added Link 7
Renamed link5.stl from openmanipulatorx to link7.stl and added it to collision and visual.

Added link7 to lite6.urdf.xacro and added links and joints to config files in the description directory

File: src/xarm_ros/xarm_description/urdf/lite6/lite6.urdf.xacro (robot description, xacro)
@@ -8,4 +8,5 @@
     joint5_lower_limit:=${-2.1642}  joint5_upper_limit:=${2.1642}
     joint6_lower_limit:=${-2.0*pi}  joint6_upper_limit:=${2.0*pi}
+    joint7_lower_limit:=${0}  joint7_upper_limit:=${0}
     model_num:=0
     inertial_params_filename:='' kinematics_params_filename:='' "
@@ -208,4 +209,33 @@
       <dynamics damping="1.0" friction="1.0"/>
     </joint>
+    <!-- ############### LINK 7 From openmanipulatorX ################### -->
+    <!-- ############### The part below may need to be recalibrated ################### -->
+    <link name="${prefix}link7">
+      <xacro:common_link_inertial
+        link_inertial_params="${inertial_params['link7']}"
+        origin_rpy="0 0 0"/>
+      <xacro:common_link_visual
+        mesh_filename="lite6/visual/link7"
+        origin_xyz="0 0 0"
+        origin_rpy="0 0 0"
+        material_name="${prefix}Silver" />
+      <xacro:common_link_collision
+        mesh_filename="lite6/collision/link7"
+        origin_xyz="0 0 0"
+        origin_rpy="0 0 0" />
+    </link>
+    <joint name="${prefix}joint7" type="fixed">
+      <!-- <origin xyz="0 0.0625 0" rpy="-1.5708 0 0" /> -->
+      <xacro:common_joint_origin joint_kinematic_params="${kinematics_params['joint7']}" />
+      <parent link="${prefix}link6" />
+      <child link="${prefix}link7" />
+      <axis xyz="0 0 1" />
+      <limit
+        lower="${joint7_lower_limit}"
+        upper="${joint7_upper_limit}"
+        effort="20.0"
+        velocity="3.14"/>
+      <dynamics damping="1.0" friction="1.0"/>
+    </joint>
     <!-- <link name="${prefix}link_eef" />
     <joint name="${prefix}joint_eef" type="fixed">

Commit message: Back to testing the fake simulation

File: src/xarm_ros/xarm_description/urdf/lite6/lite6.urdf.xacro (robot description, xacro)
@@ -8,5 +8,5 @@
     joint5_lower_limit:=${-2.1642}  joint5_upper_limit:=${2.1642}
     joint6_lower_limit:=${-2.0*pi}  joint6_upper_limit:=${2.0*pi}
-    joint7_lower_limit:=${-2.0*pi}  joint7_upper_limit:=${2.0*pi}
+    joint7_lower_limit:=${-0.010}  joint7_upper_limit:=${0.019}
     model_num:=0
     inertial_params_filename:='' kinematics_params_filename:='' "
@@ -210,4 +210,31 @@
     </joint>
     <!--############ Attach openmanipulatorX link here-->
+    <link name="${prefix}link7">
+      <xacro:common_link_inertial
+        link_inertial_params="${inertial_params['link7']}"
+        origin_rpy="0 0 0"/>
+      <xacro:common_link_visual
+        mesh_filename="lite6/visual/link7"
+        origin_xyz="0 0 0"
+        origin_rpy="0 0 0"
+        material_name="${prefix}Silver" />
+      <xacro:common_link_collision
+        mesh_filename="lite6/collision/link7"
+        origin_xyz="0 0 0"
+        origin_rpy="0 0 0" />
+    </link>
+    <joint name="${prefix}joint7" type="fixed">
+      <!-- <origin xyz="0 0.0625 0" rpy="-1.5708 0 0" /> -->
+      <xacro:common_joint_origin joint_kinematic_params="${kinematics_params['joint7']}" />
+      <parent link="${prefix}link6" />
+      <child link="${prefix}link7" />
+      <axis xyz="0 0 1" />
+      <limit
+        lower="${joint7_lower_limit}"
+        upper="${joint7_upper_limit}"
+        effort="20.0"
+        velocity="3.14"/>
+      <dynamics damping="1.0" friction="1.0"/>
+    </joint>
     <!-- <link name="${prefix}link_eef" />
     <joint name="${prefix}joint_eef" type="fixed">

File: src/xarm_ros/xarm_description/urdf/lite6/lite6_robot_macro.xacro (robot description, xacro)
@@ -37,5 +37,6 @@
           joint4_lower_limit="${-pi*0.99}" joint4_upper_limit="${pi*0.99}"
           joint5_lower_limit="${-2.1642}" joint5_upper_limit="${2.1642}"
-          joint6_lower_limit="${-pi*0.99}" joint6_upper_limit="${pi*0.99}"/>
+          joint6_lower_limit="${-pi*0.99}" joint6_upper_limit="${pi*0.99}"
+          joint7_lower_limit="${-0.010}" joint7_upper_limit="${0.019}"/>
       </xacro:if>
       <xacro:lite6_urdf prefix="${prefix}"
@@ -46,4 +47,5 @@
         joint5_lower_limit="${-2.1642}" joint5_upper_limit="${2.1642}"
         joint6_lower_limit="${-pi*0.99}" joint6_upper_limit="${pi*0.99}"
+        joint7_lower_limit="${-0.010}" joint7_upper_limit="${0.019}"
         model_num="${model_num}"
         inertial_params_filename="${inertial_params_filename}"
