Commit message: About to add the rest of the joints and links

File: src/lite6_omx/description/urdf/manipulator.urdf (robot description, URDF)
Before this commit: robot lite6_omx, 1 links, 0 joints
Links:
- removed link base_link
- added link link1; collision mesh filename=package://lite6_omx/description/meshes/collision/link1.stl; visual mesh filename=package://lite6_omx/description/meshes/visual/link1.stl
- added link link2; collision mesh filename=package://lite6_omx/description/meshes/collision/link2.stl; visual mesh filename=package://lite6_omx/description/meshes/visual/link2.stl
- added link link_base; collision mesh filename=package://lite6_omx/description/meshes/collision/link_base.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; visual mesh filename=package://lite6_omx/description/meshes/visual/link_base.stl
Joints:
- added joint joint1: type revolute, parent link_base, child link1, origin xyz=0.012 0.0 0.017 rpy=0 0 0, axis 0 0 1, limit lower=-3.142 upper=3.142 effort=1 velocity=4.8
- added joint joint2: type revolute, parent link1, child link2, origin xyz=0.012 0.0 0.017 rpy=0 0 0, axis 0 0 1, limit lower=-3.142 upper=3.142 effort=1 velocity=4.8

Commit message: Added all six links and joints from lite6

File: src/lite6_omx/description/urdf/manipulator.urdf (robot description, URDF)
Before this commit: robot lite6_omx, 3 links, 2 joints
Links:
- added link link3; collision mesh filename=package://lite6_omx/description/meshes/collision/link3.stl; visual mesh filename=package://lite6_omx/description/meshes/visual/link3.stl
- added link link4; collision mesh filename=package://lite6_omx/description/meshes/collision/link4.stl; visual mesh filename=package://lite6_omx/description/meshes/visual/link4.stl
- added link link5; collision mesh filename=package://lite6_omx/description/meshes/collision/link5.stl; visual mesh filename=package://lite6_omx/description/meshes/visual/link5.stl
- added link link6; collision mesh filename=package://lite6_omx/description/meshes/collision/link6.stl; visual mesh filename=package://lite6_omx/description/meshes/visual/link6.stl
Joints:
- added joint joint3: type revolute, parent link2, child link3, origin xyz=0.012 0.0 0.017 rpy=0 0 0, axis 0 0 1, limit lower=-3.142 upper=3.142 effort=1 velocity=4.8
- added joint joint4: type revolute, parent link3, child link4, origin xyz=0.012 0.0 0.017 rpy=0 0 0, axis 0 0 1, limit lower=-3.142 upper=3.142 effort=1 velocity=4.8
- added joint joint5: type revolute, parent link4, child link5, origin xyz=0.012 0.0 0.017 rpy=0 0 0, axis 0 0 1, limit lower=-3.142 upper=3.142 effort=1 velocity=4.8
- added joint joint6: type revolute, parent link5, child link6, origin xyz=0.012 0.0 0.017 rpy=0 0 0, axis 0 0 1, limit lower=-3.142 upper=3.142 effort=1 velocity=4.8
