Commit message: v1_scaled
Scaled but not aligned

File: src/xarm_ros/xarm_description/urdf/common/common.link.xacro (robot description, xacro)
@@ -24,16 +24,16 @@
     </xacro:unless>
   </xacro:macro>
-  <xacro:macro name="common_link_visual" params="mesh_filename add_mesh_suffix:=true material_name:='White' origin_xyz:='0 0 0' origin_rpy:='0 0 0' other_mesh_suffix:=''">
+  <xacro:macro name="common_link_visual" params="mesh_filename add_mesh_suffix:=true material_name:='White' origin_xyz:='0 0 0' origin_rpy:='0 0 0' other_mesh_suffix:='' scale:='1 1 1'">
     <visual>
       <geometry>
         <xacro:if value="${add_mesh_suffix}">
-          <mesh filename="${mesh_path}/${mesh_filename}.${mesh_suffix}"/>
+          <mesh filename="${mesh_path}/${mesh_filename}.${mesh_suffix}" scale="${scale}"/>
         </xacro:if>
         <xacro:unless value="${add_mesh_suffix}">
           <xacro:if value="${other_mesh_suffix != ''}">
-            <mesh filename="${mesh_path}/${mesh_filename}.${other_mesh_suffix}"/>
+            <mesh filename="${mesh_path}/${mesh_filename}.${other_mesh_suffix}" scale="${scale}"/>
           </xacro:if>
           <xacro:unless value="${other_mesh_suffix != ''}">
-            <mesh filename="${mesh_path}/${mesh_filename}"/>
+            <mesh filename="${mesh_path}/${mesh_filename}" scale="${scale}"/>
           </xacro:unless>
         </xacro:unless>
@@ -43,16 +43,16 @@
     </visual>
   </xacro:macro>
-  <xacro:macro name="common_link_collision" params="mesh_filename add_mesh_suffix:=true origin_xyz:='0 0 0' origin_rpy:='0 0 0' other_mesh_suffix:=''">
+  <xacro:macro name="common_link_collision" params="mesh_filename add_mesh_suffix:=true origin_xyz:='0 0 0' origin_rpy:='0 0 0' other_mesh_suffix:='' scale:='1 1 1'">
     <collision>
       <geometry>
         <xacro:if value="${add_mesh_suffix}">
-          <mesh filename="${mesh_path}/${mesh_filename}.${mesh_suffix}"/>
+          <mesh filename="${mesh_path}/${mesh_filename}.${mesh_suffix}" scale="${scale}"/>
         </xacro:if>
         <xacro:unless value="${add_mesh_suffix}">
           <xacro:if value="${other_mesh_suffix != ''}">
-            <mesh filename="${mesh_path}/${mesh_filename}.${other_mesh_suffix}"/>
+            <mesh filename="${mesh_path}/${mesh_filename}.${other_mesh_suffix}" scale="${scale}"/>
           </xacro:if>
           <xacro:unless value="${other_mesh_suffix != ''}">
-            <mesh filename="${mesh_path}/${mesh_filename}"/>
+            <mesh filename="${mesh_path}/${mesh_filename}" scale="${scale}"/>
           </xacro:unless>
         </xacro:unless>

File: src/xarm_ros/xarm_description/urdf/gripper/lite_gripper.urdf.xacro (robot description, xacro)
@@ -21,9 +21,11 @@
         origin_xyz="0 0 0"
         origin_rpy="0 0 0"
-        material_name="${prefix}White" />
+        material_name="${prefix}White"
+        scale = '0.001 0.001 0.001' />
       <xacro:common_link_collision
         mesh_filename="gripper/omx/collision/omx_gripper_base"
         origin_xyz="0 0 0"
-        origin_rpy="0 0 0" />
+        origin_rpy="0 0 0"
+        scale = '0.001 0.001 0.001' />
     </link>
     <link name="${prefix}omx_gripper_left_finger">
@@ -39,9 +41,11 @@
         origin_xyz="0 0 0"
         origin_rpy="0 0 0"
-        material_name="${prefix}White" />
+        material_name="${prefix}White"
+        scale = '0.001 0.001 0.001' />
       <xacro:common_link_collision
         mesh_filename="gripper/omx/collision/omx_left_finger"
         origin_xyz="0 0 0"
-        origin_rpy="0 0 0" />
+        origin_rpy="0 0 0"
+        scale = '0.001 0.001 0.001'/>
     </link>
     <joint name="${prefix}left_finger_joint" type="prismatic">
@@ -65,9 +69,11 @@
         origin_xyz="0 0 0"
         origin_rpy="0 0 0"
-        material_name="${prefix}White" />
+        material_name="${prefix}White"
+        scale = '0.001 0.001 0.001' />
       <xacro:common_link_collision
         mesh_filename="gripper/omx/collision/omx_right_finger"
         origin_xyz="0 0 0"
-        origin_rpy="0 0 0" />
+        origin_rpy="0 0 0"
+        scale = '0.001 0.001 0.001' />
     </link>
     <joint name="${prefix}right_finger_joint" type="prismatic">
