Commit message: Attached visuals to Robot

File: src/xarm_ros/xarm_description/urdf/gripper/lite_gripper.urdf.xacro (robot description, xacro)
@@ -10,11 +10,4 @@
     </xacro:unless>
     <link name="${prefix}uflite_gripper_link">
-      <inertial>
-        <origin xyz="0.0 0.0 0.030" rpy="0 0 0" />
-        <mass value="0.28" />
-        <inertia
-          ixx="0.00047106" ixy="3.9292E-07" ixz="2.6537E-06"
-          iyy="0.00033072" iyz="-1.0975E-05" izz="0.00025642" />
-      </inertial>
       <xacro:common_link_visual
         mesh_filename="gripper/lite/visual/gripper_lite"
@@ -24,4 +17,63 @@
       <xacro:common_link_collision
         mesh_filename="gripper/lite/collision/gripper_lite"
+        origin_xyz="0 0 0"
+        origin_rpy="0 0 0" />
+       <inertial>
+        <origin xyz="4.4206755e-02 3.6839985e-07 8.9142216e-03" />
+        <mass value="1.4327573e-01" />
+        <inertia ixx="8.0870749e-05" ixy="0.0" ixz="-1.0157896e-06"
+                 iyy="7.5980465e-05" iyz="0.0"
+                 izz="9.3127351e-05" />
+      </inertial>
+    </link>
+    <joint name="${prefix}gripper_left_joint" type="prismatic">
+      <parent link="${prefix}uflite_gripper_link"/>
+      <child link="${prefix}gripper_left_link"/>
+      <origin xyz="0.0817 0.021 0.0" rpy="0 0 0"/>
+      <axis xyz="0 1 0"/>
+      <limit velocity="4.8" effort="1" lower="-0.010" upper="0.019" />
+      <dynamics damping="0.1"/>
+    </joint>
+    <link name="${prefix}gripper_left_link">
+      <inertial>
+        <origin xyz="0 0 0" rpy="0 0 0" />
+        <mass value="1.0e-03" />
+        <inertia
+          ixx="1.0e-06" ixy="0.0" ixz="0.0"
+          iyy="1.0e-06" iyz="0.0" izz="1.0e-06" />
+      </inertial>
+      <xacro:common_link_visual
+        mesh_filename="gripper/lite/visual/gripper_left_palm"
+        origin_xyz="0 0 0"
+        origin_rpy="0 0 0"
+        material_name="${prefix}White" />
+      <xacro:common_link_collision
+        mesh_filename="gripper/lite/collision/gripper_left_palm"
+        origin_xyz="0 0 0"
+        origin_rpy="0 0 0" />
+    </link>
+    <joint name="${prefix}gripper_right_joint" type="prismatic">
+      <parent link="${prefix}uflite_gripper_link"/>
+      <child link="${prefix}gripper_right_link"/>
+      <origin xyz="0.0817 0.021 0.0" rpy="0 0 0"/>
+      <axis xyz="0 1 0"/>
+      <limit velocity="4.8" effort="1" lower="-0.010" upper="0.019" />
+      <dynamics damping="0.1"/>
+    </joint>
+     <link name="${prefix}gripper_right_link">
+      <inertial>
+        <origin xyz="0 0 0" rpy="0 0 0" />
+        <mass value="1.0e-03" />
+        <inertia
+          ixx="1.0e-06" ixy="0.0" ixz="0.0"
+          iyy="1.0e-06" iyz="0.0" izz="1.0e-06" />
+      </inertial>
+      <xacro:common_link_visual
+        mesh_filename="gripper/lite/visual/gripper_right_palm"
+        origin_xyz="0 0 0"
+        origin_rpy="0 0 0"
+        material_name="${prefix}White" />
+      <xacro:common_link_collision
+        mesh_filename="gripper/lite/collision/gripper_right_palm"
         origin_xyz="0 0 0"
         origin_rpy="0 0 0" />

File: src/xarm_ros/xarm_description/urdf/lite6/lite6.gazebo.xacro (robot description, xacro)
@@ -23,7 +23,4 @@
       <selfCollide>true</selfCollide>
     </gazebo>
-    <gazebo reference="${prefix}link7">
-      <selfCollide>true</selfCollide>
-    </gazebo>
   </xacro:macro>
 </robot>

File: src/xarm_ros/xarm_description/urdf/lite6/lite6.urdf.xacro (robot description, xacro)
@@ -8,5 +8,4 @@
     joint5_lower_limit:=${-2.1642}  joint5_upper_limit:=${2.1642}
     joint6_lower_limit:=${-2.0*pi}  joint6_upper_limit:=${2.0*pi}
-    joint7_lower_limit:=${-0.010}  joint7_upper_limit:=${0.019}
     model_num:=0
     inertial_params_filename:='' kinematics_params_filename:='' "
@@ -209,32 +208,4 @@
       <dynamics damping="1.0" friction="1.0"/>
     </joint>
-    <!--############ Attach openmanipulatorX link here-->
-    <link name="${prefix}link7">
-      <xacro:common_link_inertial
-        link_inertial_params="${inertial_params['link7']}"
-        origin_rpy="0 0 0"/>
-      <xacro:common_link_visual
-        mesh_filename="lite6/visual/link7"
-        origin_xyz="0 0 0"
-        origin_rpy="0 0 0"
-        material_name="${prefix}Silver" />
-      <xacro:common_link_collision
-        mesh_filename="lite6/collision/link7"
-        origin_xyz="0 0 0"
-        origin_rpy="0 0 0" />
-    </link>
-    <joint name="${prefix}joint7" type="fixed">
-      <!-- <origin xyz="0 0.0625 0" rpy="-1.5708 0 0" /> -->
-      <xacro:common_joint_origin joint_kinematic_params="${kinematics_params['joint7']}" />
-      <parent link="${prefix}link6" />
-      <child link="${prefix}link7" />
-      <axis xyz="0 0 1" />
-      <limit
-        lower="${joint7_lower_limit}"
-        upper="${joint7_upper_limit}"
-        effort="20.0"
-        velocity="3.14"/>
-      <dynamics damping="1.0" friction="1.0"/>
-    </joint>
     <!-- <link name="${prefix}link_eef" />
     <joint name="${prefix}joint_eef" type="fixed">

File: src/xarm_ros/xarm_description/urdf/lite6/lite6_robot_macro.xacro (robot description, xacro)
@@ -37,6 +37,5 @@
           joint4_lower_limit="${-pi*0.99}" joint4_upper_limit="${pi*0.99}"
           joint5_lower_limit="${-2.1642}" joint5_upper_limit="${2.1642}"
-          joint6_lower_limit="${-pi*0.99}" joint6_upper_limit="${pi*0.99}"
-          joint7_lower_limit="${-0.010}" joint7_upper_limit="${0.019}"/>
+          joint6_lower_limit="${-pi*0.99}" joint6_upper_limit="${pi*0.99}"/>
       </xacro:if>
       <xacro:lite6_urdf prefix="${prefix}"
@@ -47,5 +46,4 @@
         joint5_lower_limit="${-2.1642}" joint5_upper_limit="${2.1642}"
         joint6_lower_limit="${-pi*0.99}" joint6_upper_limit="${pi*0.99}"
-        joint7_lower_limit="${-0.010}" joint7_upper_limit="${0.019}"
         model_num="${model_num}"
         inertial_params_filename="${inertial_params_filename}"

Commit message: Updated urdf

File: src/xarm_ros/xarm_description/urdf/gripper/lite_gripper.urdf.xacro (robot description, xacro)
@@ -57,5 +57,5 @@
       <child link="${prefix}gripper_right_link"/>
       <origin xyz="0.0817 0.021 0.0" rpy="0 0 0"/>
-      <axis xyz="0 1 0"/>
+      <axis xyz="0 -1 0"/>
       <limit velocity="4.8" effort="1" lower="-0.010" upper="0.019" />
       <dynamics damping="0.1"/>

Commit message: Added OMX Gripper
About to make the joints movable

File: src/xarm_ros/xarm_description/urdf/gripper/lite_gripper.urdf.xacro (robot description, xacro)
@@ -5,29 +5,53 @@
       <joint name="${prefix}gripper_fix" type="fixed">
         <parent link="${attach_to}"/>
-        <child link="${prefix}uflite_gripper_link"/>
+        <child link="${prefix}omx_gripper_base_link"/>
         <origin xyz="${attach_xyz}" rpy="${attach_rpy}"/>
       </joint>
     </xacro:unless>
-    <link name="${prefix}uflite_gripper_link">
+    <!--########################### OMX Gripper Base ###########################-->
+    <link name="${prefix}omx_gripper_base_link">
+      <!--
+      <inertial>
+        <origin xyz="0.0 0.0 0.030" rpy="0 0 0" />
+        <mass value="0.28" />
+        <inertia
+          ixx="0.00047106" ixy="3.9292E-07" ixz="2.6537E-06"
+          iyy="0.00033072" iyz="-1.0975E-05" izz="0.00025642" />
+      </inertial>
+     -->
       <xacro:common_link_visual
-        mesh_filename="gripper/lite/visual/gripper_lite"
+        mesh_filename="gripper/lite/visual/omx_gripper_base"
         origin_xyz="0 0 0"
         origin_rpy="0 0 0"
         material_name="${prefix}White" />
       <xacro:common_link_collision
-        mesh_filename="gripper/lite/collision/gripper_lite"
+        mesh_filename="gripper/lite/collision/omx_gripper_base"
         origin_xyz="0 0 0"
         origin_rpy="0 0 0" />
-       <inertial>
-        <origin xyz="4.4206755e-02 3.6839985e-07 8.9142216e-03" />
-        <mass value="1.4327573e-01" />
-        <inertia ixx="8.0870749e-05" ixy="0.0" ixz="-1.0157896e-06"
-                 iyy="7.5980465e-05" iyz="0.0"
-                 izz="9.3127351e-05" />
+    </link>
+    <!--########################### OMX Gripper Left Palm ###########################-->
+    <link name="${prefix}omx_gripper_left_link">
+      <!--
+      <inertial>
+        <origin xyz="0.0 0.0 0.030" rpy="0 0 0" />
+        <mass value="0.28" />
+        <inertia
+          ixx="0.00047106" ixy="3.9292E-07" ixz="2.6537E-06"
+          iyy="0.00033072" iyz="-1.0975E-05" izz="0.00025642" />
       </inertial>
+     -->
+      <xacro:common_link_visual
+        mesh_filename="gripper/lite/visual/oxm_gripper_left_palm"
+        origin_xyz="0 0 0"
+        origin_rpy="0 0 0"
+        material_name="${prefix}Red" />
+      <xacro:common_link_collision
+        mesh_filename="gripper/lite/collision/oxm_gripper_left_palm"
+        origin_xyz="0 0 0"
+        origin_rpy="0 0 0" />
     </link>
-    <joint name="${prefix}gripper_left_joint" type="prismatic">
-      <parent link="${prefix}uflite_gripper_link"/>
-      <child link="${prefix}gripper_left_link"/>
+    <joint name="${prefix}omx_gripper_left_joint" type="prismatic">
+      <parent link="${prefix}omx_gripper_base_link"/>
+      <child link="${prefix}omx_gripper_left_link"/>
       <origin xyz="0.0817 0.021 0.0" rpy="0 0 0"/>
       <axis xyz="0 1 0"/>
@@ -35,52 +59,37 @@
       <dynamics damping="0.1"/>
     </joint>
-    <link name="${prefix}gripper_left_link">
+    <!--########################### OMX GRipper Right Palm ###########################-->
+    <link name="${prefix}omx_gripper_right_link">
+      <!--
       <inertial>
-        <origin xyz="0 0 0" rpy="0 0 0" />
-        <mass value="1.0e-03" />
+        <origin xyz="0.0 0.0 0.030" rpy="0 0 0" />
+        <mass value="0.28" />
         <inertia
-          ixx="1.0e-06" ixy="0.0" ixz="0.0"
-          iyy="1.0e-06" iyz="0.0" izz="1.0e-06" />
+          ixx="0.00047106" ixy="3.9292E-07" ixz="2.6537E-06"
+          iyy="0.00033072" iyz="-1.0975E-05" izz="0.00025642" />
       </inertial>
+     -->
       <xacro:common_link_visual
-        mesh_filename="gripper/lite/visual/gripper_left_palm"
+        mesh_filename="gripper/lite/visual/oxm_gripper_right_palm"
         origin_xyz="0 0 0"
         origin_rpy="0 0 0"
-        material_name="${prefix}White" />
+        material_name="${prefix}Black" />
       <xacro:common_link_collision
-        mesh_filename="gripper/lite/collision/gripper_left_palm"
+        mesh_filename="gripper/lite/collision/oxm_gripper_right_palm"
         origin_xyz="0 0 0"
         origin_rpy="0 0 0" />
     </link>
-    <joint name="${prefix}gripper_right_joint" type="prismatic">
-      <parent link="${prefix}uflite_gripper_link"/>
-      <child link="${prefix}gripper_right_link"/>
+    <joint name="${prefix}omx_gripper_right_joint" type="prismatic">
+      <parent link="${prefix}omx_gripper_base_link"/>
+      <child link="${prefix}omx_gripper_right_link"/>
       <origin xyz="0.0817 0.021 0.0" rpy="0 0 0"/>
-      <axis xyz="0 -1 0"/>
+      <axis xyz="0 -11 0"/>
       <limit velocity="4.8" effort="1" lower="-0.010" upper="0.019" />
       <dynamics damping="0.1"/>
     </joint>
-     <link name="${prefix}gripper_right_link">
-      <inertial>
-        <origin xyz="0 0 0" rpy="0 0 0" />
-        <mass value="1.0e-03" />
-        <inertia
-          ixx="1.0e-06" ixy="0.0" ixz="0.0"
-          iyy="1.0e-06" iyz="0.0" izz="1.0e-06" />
-      </inertial>
-      <xacro:common_link_visual
-        mesh_filename="gripper/lite/visual/gripper_right_palm"
-        origin_xyz="0 0 0"
-        origin_rpy="0 0 0"
-        material_name="${prefix}White" />
-      <xacro:common_link_collision
-        mesh_filename="gripper/lite/collision/gripper_right_palm"
-        origin_xyz="0 0 0"
-        origin_rpy="0 0 0" />
-    </link>
     <link name="${prefix}link_tcp" />
     <joint name="${prefix}joint_tcp" type="fixed">
       <origin xyz="0 0 0.0836" rpy="0 0 0" />
-      <parent link="${prefix}uflite_gripper_link" />
+      <parent link="${prefix}omx_gripper_base_link" />
       <child link="${prefix}link_tcp" />
     </joint>

Commit message: About to add left and right .stl fingers

File: src/xarm_ros/xarm_description/urdf/gripper/lite_gripper.urdf.xacro (robot description, xacro)
@@ -1,13 +1,13 @@
 <?xml version="1.0"?>
-<robot xmlns:xacro="http://ros.org/wiki/xacro" name="uflite_gripper">
+<robot xmlns:xacro="http://ros.org/wiki/xacro" name="omx_gripper">
   <xacro:macro name="uflite_gripper_urdf" params="prefix:='' attach_to:='' attach_xyz:='0 0 0' attach_rpy:='0 0 0' ">
     <xacro:unless value="${attach_to == ''}">
       <joint name="${prefix}gripper_fix" type="fixed">
         <parent link="${attach_to}"/>
-        <child link="${prefix}uflite_gripper_link"/>
+        <child link="${prefix}omx_gripper_base"/>
         <origin xyz="${attach_xyz}" rpy="${attach_rpy}"/>
       </joint>
     </xacro:unless>
-    <link name="${prefix}uflite_gripper_link">
+    <link name="${prefix}omx_gripper_base">
       <inertial>
         <origin xyz="0.0 0.0 0.030" rpy="0 0 0" />
@@ -27,5 +27,5 @@
         origin_rpy="0 0 0" />
     </link>
-  <link name="${prefix}bio_gripper_left_finger">
+    <link name="${prefix}bio_gripper_left_finger">
       <inertial>
         <origin xyz="0.021846 -0.0276 0.011911" rpy="0 0 0" />
@@ -47,5 +47,5 @@
     <joint name="${prefix}left_finger_joint" type="prismatic">
       <origin xyz="0.059 0 0.027" rpy="0 0 0" />
-      <parent link="${prefix}uflite_gripper_link" />
+      <parent link="${prefix}omx_gripper_base" />
       <child link="${prefix}bio_gripper_left_finger" />
       <axis xyz="0 1 0" />
@@ -73,5 +73,5 @@
     <joint name="${prefix}right_finger_joint" type="prismatic">
       <origin xyz="0.059 0 0.027" rpy="0 0 0" />
-      <parent link="${prefix}uflite_gripper_link" />
+      <parent link="${prefix}omx_gripper_base" />
       <child link="${prefix}bio_gripper_right_finger" />
       <axis xyz="0 1 0" />
@@ -81,5 +81,5 @@
     <joint name="${prefix}joint_tcp" type="fixed">
       <origin xyz="0 0 0.0836" rpy="0 0 0" />
-      <parent link="${prefix}uflite_gripper_link" />
+      <parent link="${prefix}omx_gripper_base" />
       <child link="${prefix}link_tcp" />
     </joint>

Commit message: Added All OMX parts
About to start calibrating the positions

File: src/xarm_ros/xarm_description/urdf/gripper/lite_gripper.urdf.xacro (robot description, xacro)
@@ -18,14 +18,14 @@
       </inertial>
       <xacro:common_link_visual
-        mesh_filename="gripper/lite/visual/omx_gripper_base"
+        mesh_filename="gripper/omx/visual/omx_gripper_base"
         origin_xyz="0 0 0"
         origin_rpy="0 0 0"
         material_name="${prefix}White" />
       <xacro:common_link_collision
-        mesh_filename="gripper/lite/collision/omx_gripper_base"
+        mesh_filename="gripper/omx/collision/omx_gripper_base"
         origin_xyz="0 0 0"
         origin_rpy="0 0 0" />
     </link>
-    <link name="${prefix}bio_gripper_left_finger">
+    <link name="${prefix}omx_gripper_left_finger">
       <inertial>
         <origin xyz="0.021846 -0.0276 0.011911" rpy="0 0 0" />
@@ -36,10 +36,10 @@
       </inertial>
       <xacro:common_link_visual
-        mesh_filename="gripper/bio/left_finger"
+        mesh_filename="gripper/omx/visual/omx_left_finger"
         origin_xyz="0 0 0"
         origin_rpy="0 0 0"
         material_name="${prefix}White" />
       <xacro:common_link_collision
-        mesh_filename="gripper/bio/left_finger"
+        mesh_filename="gripper/omx/collision/omx_left_finger"
         origin_xyz="0 0 0"
         origin_rpy="0 0 0" />
@@ -48,10 +48,10 @@
       <origin xyz="0.059 0 0.027" rpy="0 0 0" />
       <parent link="${prefix}omx_gripper_base" />
-      <child link="${prefix}bio_gripper_left_finger" />
+      <child link="${prefix}omx_gripper_left_finger" />
       <axis xyz="0 1 0" />
       <limit lower="-0.04" upper="0.0" effort="2.0" velocity="0.1" />
       <mimic joint="${prefix}right_finger_joint" multiplier="-1" offset="0" />
     </joint>
-    <link name="${prefix}bio_gripper_right_finger">
+    <link name="${prefix}omx_gripper_right_finger">
       <inertial>
         <origin xyz="0.02037 0.027565 0.010274" rpy="0 0 0" />
@@ -62,10 +62,10 @@
       </inertial>
       <xacro:common_link_visual
-        mesh_filename="gripper/bio/right_finger"
+        mesh_filename="gripper/omx/visual/omx_right_finger"
         origin_xyz="0 0 0"
         origin_rpy="0 0 0"
         material_name="${prefix}White" />
       <xacro:common_link_collision
-        mesh_filename="gripper/bio/right_finger"
+        mesh_filename="gripper/omx/collision/omx_right_finger"
         origin_xyz="0 0 0"
         origin_rpy="0 0 0" />
@@ -74,5 +74,5 @@
       <origin xyz="0.059 0 0.027" rpy="0 0 0" />
       <parent link="${prefix}omx_gripper_base" />
-      <child link="${prefix}bio_gripper_right_finger" />
+      <child link="${prefix}omx_gripper_right_finger" />
       <axis xyz="0 1 0" />
       <limit lower="0" upper="0.04" effort="2.0" velocity="0.1" />

Commit message: Renamed omx files

File: src/xarm_ros/xarm_description/urdf/gripper/lite_gripper.urdf.xacro (robot description, xacro)
@@ -5,15 +5,16 @@
       <joint name="${prefix}gripper_fix" type="fixed">
         <parent link="${attach_to}"/>
-        <child link="${prefix}omx_gripper_base"/>
+        <child link="${prefix}omx_gripper_base_link"/>
         <origin xyz="${attach_xyz}" rpy="${attach_rpy}"/>
       </joint>
     </xacro:unless>
-    <link name="${prefix}omx_gripper_base">
+    <!-- ########################### GRIPPER BASE ########################### -->
+    <link name="${prefix}omx_gripper_base_link">
       <inertial>
-        <origin xyz="0.0 0.0 0.030" rpy="0 0 0" />
-        <mass value="0.28" />
-        <inertia
-          ixx="0.00047106" ixy="3.9292E-07" ixz="2.6537E-06"
-          iyy="0.00033072" iyz="-1.0975E-05" izz="0.00025642" />
+        <origin xyz="4.4206755e-02 3.6839985e-07 8.9142216e-03" />
+        <mass value="1.4327573e-01" />
+        <inertia ixx="8.0870749e-05" ixy="0.0" ixz="-1.0157896e-06"
+                 iyy="7.5980465e-05" iyz="0.0"
+                 izz="9.3127351e-05" />
       </inertial>
       <xacro:common_link_visual
@@ -29,14 +30,15 @@
         scale = '0.001 0.001 0.001' />
     </link>
-    <link name="${prefix}omx_gripper_left_finger">
+    <!-- ########################### LEFT FINGER ########################### -->
+    <link name="${prefix}omx_gripper_left_finger_link">
       <inertial>
-        <origin xyz="0.021846 -0.0276 0.011911" rpy="0 0 0" />
-        <mass value="0.012105" />
-        <inertia
-          ixx="3.7322E-06" ixy="4.1705E-06" ixz="-4.0142E-06"
-          iyy="1.744E-05" iyz="1.2237E-06" izz="1.7775E-05" />
+        <origin xyz="0 0 0" rpy="0 0 0" />
+        <mass value="1.0e-03" />
+        <inertia ixx="1.0e-06" ixy="0.0" ixz="0.0"
+                 iyy="1.0e-06" iyz="0.0"
+                 izz="1.0e-06" />
       </inertial>
       <xacro:common_link_visual
-        mesh_filename="gripper/omx/visual/omx_left_finger"
+        mesh_filename="gripper/omx/visual/omx_gripper_left_finger"
         origin_xyz="0 0 0"
         origin_rpy="0 0 0"
@@ -44,5 +46,5 @@
         scale = '0.001 0.001 0.001' />
       <xacro:common_link_collision
-        mesh_filename="gripper/omx/collision/omx_left_finger"
+        mesh_filename="gripper/omx/collision/omx_gripper_left_finger"
         origin_xyz="0 0 0"
         origin_rpy="0 0 0"
@@ -51,20 +53,21 @@
     <joint name="${prefix}left_finger_joint" type="prismatic">
       <origin xyz="0.059 0 0.027" rpy="0 0 0" />
-      <parent link="${prefix}omx_gripper_base" />
-      <child link="${prefix}omx_gripper_left_finger" />
+      <parent link="${prefix}omx_gripper_base_link" />
+      <child link="${prefix}omx_gripper_left_finger_link" />
       <axis xyz="0 1 0" />
       <limit lower="-0.04" upper="0.0" effort="2.0" velocity="0.1" />
       <mimic joint="${prefix}right_finger_joint" multiplier="-1" offset="0" />
     </joint>
-    <link name="${prefix}omx_gripper_right_finger">
+    <!-- ########################### RIGHT FINGER ########################### -->
+    <link name="${prefix}omx_gripper_right_finger_link">
       <inertial>
-        <origin xyz="0.02037 0.027565 0.010274" rpy="0 0 0" />
-        <mass value="0.012068" />
-        <inertia
-          ixx="4.1413E-06" ixy="-3.9682E-06" ixz="-4.5734E-06"
-          iyy="1.6115E-05" iyz="-1.6711E-06" izz="1.6032E-05" />
+        <origin xyz="0 0 0" rpy="0 0 0" />
+        <mass value="1.0e-03" />
+        <inertia ixx="1.0e-06" ixy="0.0" ixz="0.0"
+                 iyy="1.0e-06" iyz="0.0"
+                 izz="1.0e-06" />
       </inertial>
       <xacro:common_link_visual
-        mesh_filename="gripper/omx/visual/omx_right_finger"
+        mesh_filename="gripper/omx/visual/omx_gripper_right_finger"
         origin_xyz="0 0 0"
         origin_rpy="0 0 0"
@@ -72,5 +75,5 @@
         scale = '0.001 0.001 0.001' />
       <xacro:common_link_collision
-        mesh_filename="gripper/omx/collision/omx_right_finger"
+        mesh_filename="gripper/omx/collision/omx_gripper_right_finger"
         origin_xyz="0 0 0"
         origin_rpy="0 0 0"
@@ -79,6 +82,6 @@
     <joint name="${prefix}right_finger_joint" type="prismatic">
       <origin xyz="0.059 0 0.027" rpy="0 0 0" />
-      <parent link="${prefix}omx_gripper_base" />
-      <child link="${prefix}omx_gripper_right_finger" />
+      <parent link="${prefix}omx_gripper_base_link" />
+      <child link="${prefix}omx_gripper_right_finger_link" />
       <axis xyz="0 1 0" />
       <limit lower="0" upper="0.04" effort="2.0" velocity="0.1" />
@@ -87,5 +90,5 @@
     <joint name="${prefix}joint_tcp" type="fixed">
       <origin xyz="0 0 0.0836" rpy="0 0 0" />
-      <parent link="${prefix}omx_gripper_base" />
+      <parent link="${prefix}omx_gripper_base_link" />
       <child link="${prefix}link_tcp" />
     </joint>
