Commit message: Completed Integration
About to resolve uflite_gripper_link warning

File: src/xarm_ros/xarm_description/urdf/gripper/lite_gripper.urdf.xacro (robot description, xacro)
@@ -52,10 +52,11 @@
     </link>
     <joint name="${prefix}left_finger_joint" type="prismatic">
-      <origin xyz="0.059 0 0.027" rpy="0 0 0" />
+      <origin xyz="0.0817 0.021 0.0" rpy="0 0 0"/>
       <parent link="${prefix}omx_gripper_base_link" />
       <child link="${prefix}omx_gripper_left_finger_link" />
       <axis xyz="0 1 0" />
-      <limit lower="-0.04" upper="0.0" effort="2.0" velocity="0.1" />
+      <limit velocity="4.8" effort="1" lower="-0.010" upper="0.019" />
       <mimic joint="${prefix}right_finger_joint" multiplier="-1" offset="0" />
+      <dynamics damping="0.1"/>
     </joint>
     <!-- ########################### RIGHT FINGER ########################### -->
@@ -81,13 +82,14 @@
     </link>
     <joint name="${prefix}right_finger_joint" type="prismatic">
-      <origin xyz="0.059 0 0.027" rpy="0 0 0" />
+      <origin xyz="0.0817 -0.021 0" rpy="0 0 0"/>
       <parent link="${prefix}omx_gripper_base_link" />
       <child link="${prefix}omx_gripper_right_finger_link" />
-      <axis xyz="0 1 0" />
-      <limit lower="0" upper="0.04" effort="2.0" velocity="0.1" />
+      <axis xyz="0 -1 0"/>
+      <limit velocity="4.8" effort="1" lower="-0.010" upper="0.019" />
+      <dynamics damping="0.1"/>
     </joint>
     <link name="${prefix}link_tcp" />
     <joint name="${prefix}joint_tcp" type="fixed">
-      <origin xyz="0 0 0.0836" rpy="0 0 0" />
+      <origin xyz="0.126 0.0 0.0" rpy="0 0 0"/>
       <parent link="${prefix}omx_gripper_base_link" />
       <child link="${prefix}link_tcp" />

Commit message: v2_integration_complete
integration complete. About to resolve collision with Gripper

File: src/xarm_ros/xarm_description/urdf/gripper/lite_gripper.urdf.xacro (robot description, xacro)
@@ -1,20 +1,20 @@
 <?xml version="1.0"?>
-<robot xmlns:xacro="http://ros.org/wiki/xacro" name="omx_gripper">
+<robot xmlns:xacro="http://ros.org/wiki/xacro" name="uflite_gripper">
   <xacro:macro name="uflite_gripper_urdf" params="prefix:='' attach_to:='' attach_xyz:='0 0 0' attach_rpy:='0 0 0' ">
     <xacro:unless value="${attach_to == ''}">
       <joint name="${prefix}gripper_fix" type="fixed">
         <parent link="${attach_to}"/>
-        <child link="${prefix}omx_gripper_base_link"/>
+        <child link="${prefix}uflite_gripper_link"/>
         <origin xyz="${attach_xyz}" rpy="${attach_rpy}"/>
       </joint>
     </xacro:unless>
     <!-- ########################### GRIPPER BASE ########################### -->
-    <link name="${prefix}omx_gripper_base_link">
+    <link name="${prefix}uflite_gripper_link">
       <inertial>
-        <origin xyz="4.4206755e-02 3.6839985e-07 8.9142216e-03" />
-        <mass value="1.4327573e-01" />
-        <inertia ixx="8.0870749e-05" ixy="0.0" ixz="-1.0157896e-06"
-                 iyy="7.5980465e-05" iyz="0.0"
-                 izz="9.3127351e-05" />
+        <origin xyz="0.0 0.0 0.030" rpy="0 0 0" />
+        <mass value="0.28" />
+        <inertia
+          ixx="0.00047106" ixy="3.9292E-07" ixz="2.6537E-06"
+          iyy="0.00033072" iyz="-1.0975E-05" izz="0.00025642" />
       </inertial>
       <xacro:common_link_visual
@@ -53,5 +53,5 @@
     <joint name="${prefix}left_finger_joint" type="prismatic">
       <origin xyz="0.0817 0.021 0.0" rpy="0 0 0"/>
-      <parent link="${prefix}omx_gripper_base_link" />
+      <parent link="${prefix}uflite_gripper_link" />
       <child link="${prefix}omx_gripper_left_finger_link" />
       <axis xyz="0 1 0" />
@@ -83,5 +83,5 @@
     <joint name="${prefix}right_finger_joint" type="prismatic">
       <origin xyz="0.0817 -0.021 0" rpy="0 0 0"/>
-      <parent link="${prefix}omx_gripper_base_link" />
+      <parent link="${prefix}uflite_gripper_link" />
       <child link="${prefix}omx_gripper_right_finger_link" />
       <axis xyz="0 -1 0"/>
@@ -92,5 +92,5 @@
     <joint name="${prefix}joint_tcp" type="fixed">
       <origin xyz="0.126 0.0 0.0" rpy="0 0 0"/>
-      <parent link="${prefix}omx_gripper_base_link" />
+      <parent link="${prefix}uflite_gripper_link" />
       <child link="${prefix}link_tcp" />
     </joint>

Commit message: no_collision
no collision but needs offset

File: src/xarm_ros/xarm_description/urdf/gripper/lite_gripper.urdf.xacro (robot description, xacro)
@@ -11,15 +11,15 @@
     <!-- ########################### GRIPPER BASE ########################### -->
     <link name="${prefix}uflite_gripper_link">
-      <inertial>
-        <origin xyz="0.0 0.0 0.030" rpy="0 0 0" />
-        <mass value="0.28" />
-        <inertia
-          ixx="0.00047106" ixy="3.9292E-07" ixz="2.6537E-06"
-          iyy="0.00033072" iyz="-1.0975E-05" izz="0.00025642" />
+       <inertial>
+        <origin xyz="4.4206755e-02 3.6839985e-07 8.9142216e-03" />
+        <mass value="1.4327573e-01" />
+        <inertia ixx="8.0870749e-05" ixy="0.0" ixz="-1.0157896e-06"
+                 iyy="7.5980465e-05" iyz="0.0"
+                 izz="9.3127351e-05" />
       </inertial>
       <xacro:common_link_visual
         mesh_filename="gripper/omx/visual/omx_gripper_base"
         origin_xyz="0 0 0"
-        origin_rpy="0 0 0"
+        origin_rpy="0 -1.5708 0"
         material_name="${prefix}White"
         scale = '0.001 0.001 0.001' />
@@ -27,5 +27,5 @@
         mesh_filename="gripper/omx/collision/omx_gripper_base"
         origin_xyz="0 0 0"
-        origin_rpy="0 0 0"
+        origin_rpy="0 -1.5708  0"
         scale = '0.001 0.001 0.001' />
     </link>
@@ -42,5 +42,5 @@
         mesh_filename="gripper/omx/visual/omx_gripper_left_finger"
         origin_xyz="0 0 0"
-        origin_rpy="0 0 0"
+        origin_rpy="0 -1.5708 0"
         material_name="${prefix}White"
         scale = '0.001 0.001 0.001' />
@@ -48,5 +48,5 @@
         mesh_filename="gripper/omx/collision/omx_gripper_left_finger"
         origin_xyz="0 0 0"
-        origin_rpy="0 0 0"
+        origin_rpy="0 -1.5708 0"
         scale = '0.001 0.001 0.001'/>
     </link>
@@ -72,5 +72,5 @@
         mesh_filename="gripper/omx/visual/omx_gripper_right_finger"
         origin_xyz="0 0 0"
-        origin_rpy="0 0 0"
+        origin_rpy="0 -1.5708  0"
         material_name="${prefix}White"
         scale = '0.001 0.001 0.001' />
@@ -78,5 +78,5 @@
         mesh_filename="gripper/omx/collision/omx_gripper_right_finger"
         origin_xyz="0 0 0"
-        origin_rpy="0 0 0"
+        origin_rpy="0 -1.5708  0"
         scale = '0.001 0.001 0.001' />
     </link>

Commit message: aligned with collision
aligned but with collision

File: src/xarm_ros/xarm_description/urdf/gripper/lite_gripper.urdf.xacro (robot description, xacro)
@@ -52,5 +52,5 @@
     </link>
     <joint name="${prefix}left_finger_joint" type="prismatic">
-      <origin xyz="0.0817 0.021 0.0" rpy="0 0 0"/>
+      <origin xyz="0.0 0.021 0.0817" rpy="0 0 0"/>
       <parent link="${prefix}uflite_gripper_link" />
       <child link="${prefix}omx_gripper_left_finger_link" />
@@ -82,5 +82,5 @@
     </link>
     <joint name="${prefix}right_finger_joint" type="prismatic">
-      <origin xyz="0.0817 -0.021 0" rpy="0 0 0"/>
+      <origin xyz="0.0 -0.021 0.0817" rpy="0 0 0"/>
       <parent link="${prefix}uflite_gripper_link" />
       <child link="${prefix}omx_gripper_right_finger_link" />

Commit message: No collision but not aligned with robot

File: src/xarm_ros/xarm_description/urdf/gripper/lite_gripper.urdf.xacro (robot description, xacro)
@@ -21,5 +21,5 @@
         mesh_filename="gripper/omx/visual/omx_gripper_base"
         origin_xyz="0 0 0"
-        origin_rpy="0 -1.5708 3.14159"
+        origin_rpy="0 -1.5708 0"
         material_name="${prefix}White"
         scale = '0.001 0.001 0.001' />
@@ -27,5 +27,5 @@
         mesh_filename="gripper/omx/collision/omx_gripper_base"
         origin_xyz="0 0 0"
-        origin_rpy="0 -1.5708  3.14159"
+        origin_rpy="0 -1.5708  0"
         scale = '0.001 0.001 0.001' />
     </link>
@@ -42,5 +42,5 @@
         mesh_filename="gripper/omx/visual/omx_gripper_left_finger"
         origin_xyz="0 0 0"
-        origin_rpy="0 -1.5708 0"
+        origin_rpy="0 0 0"
         material_name="${prefix}White"
         scale = '0.001 0.001 0.001' />
@@ -48,9 +48,9 @@
         mesh_filename="gripper/omx/collision/omx_gripper_left_finger"
         origin_xyz="0 0 0"
-        origin_rpy="0 -1.5708 0"
+        origin_rpy="0 0 0"
         scale = '0.001 0.001 0.001'/>
     </link>
     <joint name="${prefix}left_finger_joint" type="prismatic">
-      <origin xyz="0.0 0.021 0.0817" rpy="0 0 0"/>
+      <origin xyz="0.0817 0.021 0.0" rpy="0 0 0"/>
       <parent link="${prefix}uflite_gripper_link" />
       <child link="${prefix}omx_gripper_left_finger_link" />
@@ -72,5 +72,5 @@
         mesh_filename="gripper/omx/visual/omx_gripper_right_finger"
         origin_xyz="0 0 0"
-        origin_rpy="0 -1.5708  0"
+        origin_rpy="0 0 0"
         material_name="${prefix}White"
         scale = '0.001 0.001 0.001' />
@@ -78,9 +78,9 @@
         mesh_filename="gripper/omx/collision/omx_gripper_right_finger"
         origin_xyz="0 0 0"
-        origin_rpy="0 -1.5708  0"
+        origin_rpy="0 0 0"
         scale = '0.001 0.001 0.001' />
     </link>
     <joint name="${prefix}right_finger_joint" type="prismatic">
-      <origin xyz="0.0 -0.021 0.0817" rpy="0 0 0"/>
+      <origin xyz="0.0817 -0.021 0" rpy="0 0 0"/>
       <parent link="${prefix}uflite_gripper_link" />
       <child link="${prefix}omx_gripper_right_finger_link" />

Commit message: Proper bubble and orientation but with collision
TODO: Fix collision

File: src/xarm_ros/xarm_description/urdf/gripper/lite_gripper.urdf.xacro (robot description, xacro)
@@ -42,5 +42,5 @@
         mesh_filename="gripper/omx/visual/omx_gripper_left_finger"
         origin_xyz="0 0 0"
-        origin_rpy="0 0 0"
+        origin_rpy="0 -1.5708 0"
         material_name="${prefix}White"
         scale = '0.001 0.001 0.001' />
@@ -48,9 +48,9 @@
         mesh_filename="gripper/omx/collision/omx_gripper_left_finger"
         origin_xyz="0 0 0"
-        origin_rpy="0 0 0"
+        origin_rpy="0 -1.5708 0"
         scale = '0.001 0.001 0.001'/>
     </link>
     <joint name="${prefix}left_finger_joint" type="prismatic">
-      <origin xyz="0.0817 0.021 0.0" rpy="0 0 0"/>
+      <origin xyz="0.0 0.021 0.0817" rpy="0 0 0"/>
       <parent link="${prefix}uflite_gripper_link" />
       <child link="${prefix}omx_gripper_left_finger_link" />
@@ -72,5 +72,5 @@
         mesh_filename="gripper/omx/visual/omx_gripper_right_finger"
         origin_xyz="0 0 0"
-        origin_rpy="0 0 0"
+        origin_rpy="0 -1.5708  0"
         material_name="${prefix}White"
         scale = '0.001 0.001 0.001' />
@@ -78,9 +78,9 @@
         mesh_filename="gripper/omx/collision/omx_gripper_right_finger"
         origin_xyz="0 0 0"
-        origin_rpy="0 0 0"
+        origin_rpy="0 -1.5708  0"
         scale = '0.001 0.001 0.001' />
     </link>
     <joint name="${prefix}right_finger_joint" type="prismatic">
-      <origin xyz="0.0817 -0.021 0" rpy="0 0 0"/>
+      <origin xyz="0.0 -0.021 0.0817" rpy="0 0 0"/>
       <parent link="${prefix}uflite_gripper_link" />
       <child link="${prefix}omx_gripper_right_finger_link" />
@@ -91,5 +91,5 @@
     <link name="${prefix}link_tcp" />
     <joint name="${prefix}joint_tcp" type="fixed">
-      <origin xyz="0.126 0.0 0.0" rpy="0 0 0"/>
+      <origin xyz="0 0.0 0.126" rpy="0 0 0"/>
       <parent link="${prefix}uflite_gripper_link" />
       <child link="${prefix}link_tcp" />

Commit message: Added coupler

File: src/xarm_ros/xarm_description/urdf/gripper/lite_gripper.urdf.xacro (robot description, xacro)
@@ -11,5 +11,5 @@
     <!-- ########################### GRIPPER BASE ########################### -->
     <link name="${prefix}uflite_gripper_link">
-       <inertial>
+      <inertial>
         <origin xyz="4.4206755e-02 3.6839985e-07 8.9142216e-03" />
         <mass value="1.4327573e-01" />
@@ -18,4 +18,18 @@
                  izz="9.3127351e-05" />
       </inertial>
+      <!-- Coupler Visual -->
+      <xacro:common_link_visual
+        mesh_filename="gripper/omx/visual/coupler"
+        origin_xyz="0 0 0"
+        origin_rpy="0 0 0"
+        material_name="${prefix}White"
+        scale='0.001 0.001 0.001' />
+      <!-- Coupler Collision -->
+      <xacro:common_link_collision
+        mesh_filename="gripper/omx/collision/coupler"
+        origin_xyz="0 0 0"
+        origin_rpy="0 0 0"
+        scale='0.001 0.001 0.001' />
+      <!-- Gripper Base Visual -->
       <xacro:common_link_visual
         mesh_filename="gripper/omx/visual/omx_gripper_base"
@@ -23,10 +37,11 @@
         origin_rpy="0 -1.5708 0"
         material_name="${prefix}White"
-        scale = '1 1 1' />
+        scale="1 1 1" />
+      <!-- Gripper Base Collision -->
       <xacro:common_link_collision
         mesh_filename="gripper/omx/collision/omx_gripper_base"
         origin_xyz="0 0 0"
         origin_rpy="0 0 0"
-        scale = '1 1 1' />
+        scale="1 1 1" />
     </link>
     <!-- ########################### LEFT FINGER ########################### -->

Commit message: About to set origin of pincers to 0

File: src/xarm_ros/xarm_description/urdf/gripper/lite_gripper.urdf.xacro (robot description, xacro)
@@ -12,9 +12,9 @@
     <link name="${prefix}uflite_gripper_link">
       <inertial>
-        <origin xyz="4.4206755e-02 3.6839985e-07 8.9142216e-03" />
-        <mass value="1.4327573e-01" />
-        <inertia ixx="8.0870749e-05" ixy="0.0" ixz="-1.0157896e-06"
-                 iyy="7.5980465e-05" iyz="0.0"
-                 izz="9.3127351e-05" />
+        <origin xyz="0 0 0" rpy="0 0 0" />
+        <mass value="1.0e-03" />
+        <inertia ixx="1.0e-06" ixy="0.0" ixz="0.0"
+                 iyy="1.0e-06" iyz="0.0"
+                 izz="1.0e-06" />
       </inertial>
       <!-- Coupler Visual -->

Commit message: v5_rough_alignment
Version 5 roughly aligned

File: src/xarm_ros/xarm_description/urdf/gripper/lite_gripper.urdf.xacro (robot description, xacro)
@@ -50,5 +50,5 @@
     <link name="${prefix}omx_gripper_left_finger_link">
       <inertial>
-        <origin xyz="0 0 0" rpy="0 0 0" />
+        <origin xyz="0 0 -0.0191" rpy="0 0 0" />
         <mass value="1.0e-03" />
         <inertia ixx="1.0e-06" ixy="0.0" ixz="0.0"
@@ -58,5 +58,5 @@
       <xacro:common_link_visual
         mesh_filename="gripper/omx/visual/omx_gripper_left_finger"
-        origin_xyz="0 0 0"
+        origin_xyz="0 0 -0.0191"
         origin_rpy="0 -1.5708 0"
         material_name="${prefix}White"
@@ -64,5 +64,5 @@
       <xacro:common_link_collision
         mesh_filename="gripper/omx/collision/omx_gripper_left_finger"
-        origin_xyz="0 0 0"
+        origin_xyz="0 0 -0.0191"
         origin_rpy="0 -1.5708 0"
         scale = '0.001 0.001 0.001'/>
@@ -80,5 +80,5 @@
     <link name="${prefix}omx_gripper_right_finger_link">
       <inertial>
-        <origin xyz="0 0 0" rpy="0 0 0" />
+        <origin xyz="0 0 -0.0191" rpy="0 0 0" />
         <mass value="1.0e-03" />
         <inertia ixx="1.0e-06" ixy="0.0" ixz="0.0"
@@ -88,5 +88,5 @@
       <xacro:common_link_visual
         mesh_filename="gripper/omx/visual/omx_gripper_right_finger"
-        origin_xyz="0 0 0"
+        origin_xyz="0 0 -0.0191"
         origin_rpy="0 -1.5708  0"
         material_name="${prefix}White"
@@ -94,5 +94,5 @@
       <xacro:common_link_collision
         mesh_filename="gripper/omx/collision/omx_gripper_right_finger"
-        origin_xyz="0 0 0"
+        origin_xyz="0 0 -0.0191"
         origin_rpy="0 -1.5708  0"
         scale = '0.001 0.001 0.001' />

Commit message: Added a joint between a coupler and gripper base link

File: src/xarm_ros/xarm_description/urdf/gripper/lite_gripper.urdf.xacro (robot description, xacro)
@@ -9,5 +9,5 @@
       </joint>
     </xacro:unless>
-    <!-- ########################### GRIPPER BASE ########################### -->
+    <!-- ########################### MAIN GRIPPER BASE LINK ########################### -->
     <link name="${prefix}uflite_gripper_link">
       <inertial>
@@ -18,19 +18,4 @@
                  izz="1.0e-06" />
       </inertial>
-      <!-- ########################### COUPLER  ########################### -->
-      <!-- Coupler Visual -->
-      <xacro:common_link_visual
-        mesh_filename="gripper/omx/visual/coupler"
-        origin_xyz="0 0 0.01491"
-        origin_rpy="0 -3.14159 0"
-        material_name="${prefix}White"
-        scale='0.001 0.001 0.001' />
-      <!-- Coupler Collision -->
-      <xacro:common_link_collision
-        mesh_filename="gripper/omx/collision/coupler"
-        origin_xyz="0 0 0.01491"
-        origin_rpy="0 -3.14159 0"
-        scale="0.001 0.001 0.001" />
-       <!-- ########################### BASE LINK  ########################### -->
       <!-- Gripper Base Visual -->
       <xacro:common_link_visual
@@ -47,4 +32,30 @@
         scale="1 1 1" />
     </link>
+    <!-- ########################### COUPLER SEPARATE LINK ########################### -->
+    <link name="${prefix}uflite_gripper_coupler_link">
+      <inertial>
+        <origin xyz="0 0 0" rpy="0 0 0" />
+        <mass value="1.0e-03" />
+        <inertia ixx="1.0e-06" ixy="0.0" ixz="0.0"
+                 iyy="1.0e-06" iyz="0.0"
+                 izz="1.0e-06" />
+      </inertial>
+      <xacro:common_link_visual
+        mesh_filename="gripper/omx/visual/coupler"
+        origin_xyz="0 0 0.01491"
+        origin_rpy="0 -3.14159 0"
+        material_name="${prefix}White"
+        scale='0.001 0.001 0.001' />
+      <xacro:common_link_collision
+        mesh_filename="gripper/omx/collision/coupler"
+        origin_xyz="0 0 0.01491"
+        origin_rpy="0 -3.14159 0"
+        scale="0.001 0.001 0.001" />
+    </link>
+    <joint name="${prefix}gripper_coupler_fixed" type="fixed">
+      <parent link="${prefix}uflite_gripper_link" />
+      <child link="${prefix}uflite_gripper_coupler_link" />
+      <origin xyz="0 0 0" rpy="0 0 0" />
+    </joint>
     <!-- ########################### LEFT FINGER ########################### -->
     <link name="${prefix}omx_gripper_left_finger_link">
@@ -106,4 +117,5 @@
       <dynamics damping="0.1"/>
     </joint>
+    <!-- ########################### TCP ########################### -->
     <link name="${prefix}link_tcp" />
     <joint name="${prefix}joint_tcp" type="fixed">

Commit message: About to fix bounding boxed

File: src/xarm_ros/xarm_description/urdf/gripper/lite_gripper.urdf.xacro (robot description, xacro)
@@ -9,4 +9,30 @@
       </joint>
     </xacro:unless>
+    <!-- ########################### COUPLER SEPARATE LINK ########################### -->
+    <link name="${prefix}uflite_gripper_coupler_link">
+      <inertial>
+        <origin xyz="0 0 0" rpy="0 0 0" />
+        <mass value="1.0e-03" />
+        <inertia ixx="1.0e-06" ixy="0.0" ixz="0.0"
+                 iyy="1.0e-06" iyz="0.0"
+                 izz="1.0e-06" />
+      </inertial>
+      <xacro:common_link_visual
+        mesh_filename="gripper/omx/visual/coupler"
+        origin_xyz="0 0 0.015"
+        origin_rpy="0 -3.14159 0"
+        material_name="${prefix}White"
+        scale='0.001 0.001 0.001' />
+      <xacro:common_link_collision
+        mesh_filename="gripper/omx/collision/coupler"
+        origin_xyz="0 0 0.015"
+        origin_rpy="0 -3.14159 0"
+        scale="0.001 0.001 0.001" />
+    </link>
+    <joint name="${prefix}gripper_coupler_fixed" type="fixed">
+      <parent link="${prefix}uflite_gripper_link" />
+      <child link="${prefix}uflite_gripper_coupler_link" />
+      <origin xyz="0 0 0" rpy="0 0 0" />
+    </joint>
     <!-- ########################### MAIN GRIPPER BASE LINK ########################### -->
     <link name="${prefix}uflite_gripper_link">
@@ -32,30 +58,4 @@
         scale="1 1 1" />
     </link>
-    <!-- ########################### COUPLER SEPARATE LINK ########################### -->
-    <link name="${prefix}uflite_gripper_coupler_link">
-      <inertial>
-        <origin xyz="0 0 0" rpy="0 0 0" />
-        <mass value="1.0e-03" />
-        <inertia ixx="1.0e-06" ixy="0.0" ixz="0.0"
-                 iyy="1.0e-06" iyz="0.0"
-                 izz="1.0e-06" />
-      </inertial>
-      <xacro:common_link_visual
-        mesh_filename="gripper/omx/visual/coupler"
-        origin_xyz="0 0 0.01491"
-        origin_rpy="0 -3.14159 0"
-        material_name="${prefix}White"
-        scale='0.001 0.001 0.001' />
-      <xacro:common_link_collision
-        mesh_filename="gripper/omx/collision/coupler"
-        origin_xyz="0 0 0.01491"
-        origin_rpy="0 -3.14159 0"
-        scale="0.001 0.001 0.001" />
-    </link>
-    <joint name="${prefix}gripper_coupler_fixed" type="fixed">
-      <parent link="${prefix}uflite_gripper_link" />
-      <child link="${prefix}uflite_gripper_coupler_link" />
-      <origin xyz="0 0 0" rpy="0 0 0" />
-    </joint>
     <!-- ########################### LEFT FINGER ########################### -->
     <link name="${prefix}omx_gripper_left_finger_link">
