Commit message: fixed coupler

File: src/xarm_ros/xarm_description/urdf/gripper/lite_gripper.urdf.xacro (robot description, xacro)
@@ -12,13 +12,13 @@
     <link name="${prefix}uflite_gripper_coupler_link">
       <inertial>
-        <origin xyz="0 0 0" rpy="0 0 0" />
-        <mass value="1.0e-03" />
-        <inertia ixx="1.0e-06" ixy="0.0" ixz="0.0"
-                 iyy="1.0e-06" iyz="0.0"
-                 izz="1.0e-06" />
+        <origin xyz="0.0 0.0 0.030" rpy="0 0 0" />
+        <mass value="0.28" />
+        <inertia
+          ixx="0.00047106" ixy="3.9292E-07" ixz="2.6537E-06"
+          iyy="0.00033072" iyz="-1.0975E-05" izz="0.00025642" />
       </inertial>
       <xacro:common_link_visual
         mesh_filename="gripper/omx/visual/coupler"
-        origin_xyz="0 0 0.025"
+        origin_xyz="0 0 0.015"
         origin_rpy="0 -3.14159 0"
         material_name="${prefix}White"
@@ -26,5 +26,5 @@
       <xacro:common_link_collision
         mesh_filename="gripper/omx/collision/coupler"
-        origin_xyz="0 0 0.025"
+        origin_xyz="0 0 0.015"
         origin_rpy="0 -3.14159 0"
         scale="0.001 0.001 0.001" />
@@ -61,5 +61,5 @@
     <link name="${prefix}omx_gripper_left_finger_link">
       <inertial>
-        <origin xyz="0 0 -0.0191" rpy="0 0 0" />
+        <origin xyz="0 0 0.5" rpy="0 0 0" />
         <mass value="1.0e-03" />
         <inertia ixx="1.0e-06" ixy="0.0" ixz="0.0"
@@ -69,5 +69,5 @@
       <xacro:common_link_visual
         mesh_filename="gripper/omx/visual/omx_gripper_left_finger"
-        origin_xyz="0 0 -0.0191"
+        origin_xyz="0 0 0.5"
         origin_rpy="0 -1.5708 0"
         material_name="${prefix}White"
@@ -75,5 +75,5 @@
       <xacro:common_link_collision
         mesh_filename="gripper/omx/collision/omx_gripper_left_finger"
-        origin_xyz="0 0 -0.0191"
+        origin_xyz="0 0 0.5"
         origin_rpy="0 -1.5708 0"
         scale = '0.001 0.001 0.001'/>
@@ -91,5 +91,5 @@
     <link name="${prefix}omx_gripper_right_finger_link">
       <inertial>
-        <origin xyz="0 0 -0.0191" rpy="0 0 0" />
+        <origin xyz="0 0 0.5" rpy="0 0 0" />
         <mass value="1.0e-03" />
         <inertia ixx="1.0e-06" ixy="0.0" ixz="0.0"
@@ -99,5 +99,5 @@
       <xacro:common_link_visual
         mesh_filename="gripper/omx/visual/omx_gripper_right_finger"
-        origin_xyz="0 0 -0.0191"
+        origin_xyz="0 0 0.5"
         origin_rpy="0 -1.5708  0"
         material_name="${prefix}White"
@@ -105,5 +105,5 @@
       <xacro:common_link_collision
         mesh_filename="gripper/omx/collision/omx_gripper_right_finger"
-        origin_xyz="0 0 -0.0191"
+        origin_xyz="0 0 0.5"
         origin_rpy="0 -1.5708  0"
         scale = '0.001 0.001 0.001' />

Commit message: Completed Alignment in URDF

File: src/xarm_ros/xarm_description/urdf/gripper/lite_gripper.urdf.xacro (robot description, xacro)
@@ -61,5 +61,5 @@
     <link name="${prefix}omx_gripper_left_finger_link">
       <inertial>
-        <origin xyz="0 0 0.5" rpy="0 0 0" />
+        <origin xyz="0 0 -0.01679" rpy="0 0 0" />
         <mass value="1.0e-03" />
         <inertia ixx="1.0e-06" ixy="0.0" ixz="0.0"
@@ -69,5 +69,5 @@
       <xacro:common_link_visual
         mesh_filename="gripper/omx/visual/omx_gripper_left_finger"
-        origin_xyz="0 0 0.5"
+        origin_xyz="0 0 -0.01679"
         origin_rpy="0 -1.5708 0"
         material_name="${prefix}White"
@@ -75,5 +75,5 @@
       <xacro:common_link_collision
         mesh_filename="gripper/omx/collision/omx_gripper_left_finger"
-        origin_xyz="0 0 0.5"
+        origin_xyz="0 0 -0.01679"
         origin_rpy="0 -1.5708 0"
         scale = '0.001 0.001 0.001'/>
@@ -91,5 +91,5 @@
     <link name="${prefix}omx_gripper_right_finger_link">
       <inertial>
-        <origin xyz="0 0 0.5" rpy="0 0 0" />
+        <origin xyz="0 0 -0.01679" rpy="0 0 0" />
         <mass value="1.0e-03" />
         <inertia ixx="1.0e-06" ixy="0.0" ixz="0.0"
@@ -99,5 +99,5 @@
       <xacro:common_link_visual
         mesh_filename="gripper/omx/visual/omx_gripper_right_finger"
-        origin_xyz="0 0 0.5"
+        origin_xyz="0 0 -0.01679"
         origin_rpy="0 -1.5708  0"
         material_name="${prefix}White"
@@ -105,5 +105,5 @@
       <xacro:common_link_collision
         mesh_filename="gripper/omx/collision/omx_gripper_right_finger"
-        origin_xyz="0 0 0.5"
+        origin_xyz="0 0 -0.01679"
         origin_rpy="0 -1.5708  0"
         scale = '0.001 0.001 0.001' />

Commit message: fixed collion between link6 and coupler

File: src/xarm_ros/xarm_description/urdf/gripper/lite_gripper.urdf.xacro (robot description, xacro)
@@ -20,5 +20,5 @@
       <xacro:common_link_visual
         mesh_filename="gripper/omx/visual/coupler"
-        origin_xyz="0 0 0.015"
+        origin_xyz="0 0 0.01501"
         origin_rpy="0 -3.14159 0"
         material_name="${prefix}White"
@@ -26,5 +26,5 @@
       <xacro:common_link_collision
         mesh_filename="gripper/omx/collision/coupler"
-        origin_xyz="0 0 0.015"
+        origin_xyz="0 0 0.01501"
         origin_rpy="0 -3.14159 0"
         scale="0.001 0.001 0.001" />
@@ -47,5 +47,5 @@
       <xacro:common_link_visual
         mesh_filename="gripper/omx/visual/omx_gripper_base"
-        origin_xyz="0.2101 0 -0.145"
+        origin_xyz="0.2101 0 0.3"
         origin_rpy="0 -1.5708 0"
         material_name="${prefix}White"
@@ -54,5 +54,5 @@
       <xacro:common_link_collision
         mesh_filename="gripper/omx/collision/omx_gripper_base"
-        origin_xyz="0.2101 0 -0.145"
+        origin_xyz="0.2101 0 0.3"
         origin_rpy="0 -1.5708 0"
         scale="1 1 1" />
@@ -61,5 +61,5 @@
     <link name="${prefix}omx_gripper_left_finger_link">
       <inertial>
-        <origin xyz="0 0 -0.01679" rpy="0 0 0" />
+        <origin xyz="0 0 0.5" rpy="0 0 0" />
         <mass value="1.0e-03" />
         <inertia ixx="1.0e-06" ixy="0.0" ixz="0.0"
@@ -69,5 +69,5 @@
       <xacro:common_link_visual
         mesh_filename="gripper/omx/visual/omx_gripper_left_finger"
-        origin_xyz="0 0 -0.01679"
+        origin_xyz="0 0 0.5"
         origin_rpy="0 -1.5708 0"
         material_name="${prefix}White"
@@ -75,5 +75,5 @@
       <xacro:common_link_collision
         mesh_filename="gripper/omx/collision/omx_gripper_left_finger"
-        origin_xyz="0 0 -0.01679"
+        origin_xyz="0 0 0.5"
         origin_rpy="0 -1.5708 0"
         scale = '0.001 0.001 0.001'/>
@@ -91,5 +91,5 @@
     <link name="${prefix}omx_gripper_right_finger_link">
       <inertial>
-        <origin xyz="0 0 -0.01679" rpy="0 0 0" />
+        <origin xyz="0 0 0.5" rpy="0 0 0" />
         <mass value="1.0e-03" />
         <inertia ixx="1.0e-06" ixy="0.0" ixz="0.0"
@@ -99,5 +99,5 @@
       <xacro:common_link_visual
         mesh_filename="gripper/omx/visual/omx_gripper_right_finger"
-        origin_xyz="0 0 -0.01679"
+        origin_xyz="0 0 0.5"
         origin_rpy="0 -1.5708  0"
         material_name="${prefix}White"
@@ -105,5 +105,5 @@
       <xacro:common_link_collision
         mesh_filename="gripper/omx/collision/omx_gripper_right_finger"
-        origin_xyz="0 0 -0.01679"
+        origin_xyz="0 0 0.5"
         origin_rpy="0 -1.5708  0"
         scale = '0.001 0.001 0.001' />

Commit message: fixed visiual fit between gripper_base and coupler

File: src/xarm_ros/xarm_description/urdf/gripper/lite_gripper.urdf.xacro (robot description, xacro)
@@ -12,5 +12,5 @@
     <link name="${prefix}uflite_gripper_coupler_link">
       <inertial>
-        <origin xyz="0.0 0.0 0.030" rpy="0 0 0" />
+        <origin xyz="0.0 0.0 0.0" rpy="0 0 0" />
         <mass value="0.28" />
         <inertia
@@ -38,5 +38,5 @@
     <link name="${prefix}uflite_gripper_link">
       <inertial>
-        <origin xyz="0 0 0" rpy="0 0 0" />
+        <origin xyz="0 0 -0.141" rpy="0 0 0" />
         <mass value="1.0e-03" />
         <inertia ixx="1.0e-06" ixy="0.0" ixz="0.0"
@@ -47,5 +47,5 @@
       <xacro:common_link_visual
         mesh_filename="gripper/omx/visual/omx_gripper_base"
-        origin_xyz="0.2101 0 0.3"
+        origin_xyz="0.2101 0 -0.141"
         origin_rpy="0 -1.5708 0"
         material_name="${prefix}White"
@@ -54,5 +54,5 @@
       <xacro:common_link_collision
         mesh_filename="gripper/omx/collision/omx_gripper_base"
-        origin_xyz="0.2101 0 0.3"
+        origin_xyz="0.2101 0 -0.141"
         origin_rpy="0 -1.5708 0"
         scale="1 1 1" />

Commit message: fixed visuals in the gripper fingers

File: src/xarm_ros/xarm_description/urdf/gripper/lite_gripper.urdf.xacro (robot description, xacro)
@@ -61,5 +61,5 @@
     <link name="${prefix}omx_gripper_left_finger_link">
       <inertial>
-        <origin xyz="0 0 0.5" rpy="0 0 0" />
+        <origin xyz="0 0 0" rpy="0 0 0" />
         <mass value="1.0e-03" />
         <inertia ixx="1.0e-06" ixy="0.0" ixz="0.0"
@@ -69,5 +69,5 @@
       <xacro:common_link_visual
         mesh_filename="gripper/omx/visual/omx_gripper_left_finger"
-        origin_xyz="0 0 0.5"
+        origin_xyz="0 0 -0.01368"
         origin_rpy="0 -1.5708 0"
         material_name="${prefix}White"
@@ -75,5 +75,5 @@
       <xacro:common_link_collision
         mesh_filename="gripper/omx/collision/omx_gripper_left_finger"
-        origin_xyz="0 0 0.5"
+        origin_xyz="0 0 -0.01368"
         origin_rpy="0 -1.5708 0"
         scale = '0.001 0.001 0.001'/>
@@ -91,5 +91,5 @@
     <link name="${prefix}omx_gripper_right_finger_link">
       <inertial>
-        <origin xyz="0 0 0.5" rpy="0 0 0" />
+        <origin xyz="0 0 0" rpy="0 0 0" />
         <mass value="1.0e-03" />
         <inertia ixx="1.0e-06" ixy="0.0" ixz="0.0"
@@ -99,5 +99,5 @@
       <xacro:common_link_visual
         mesh_filename="gripper/omx/visual/omx_gripper_right_finger"
-        origin_xyz="0 0 0.5"
+        origin_xyz="0 0 -0.01368"
         origin_rpy="0 -1.5708  0"
         material_name="${prefix}White"
@@ -105,5 +105,5 @@
       <xacro:common_link_collision
         mesh_filename="gripper/omx/collision/omx_gripper_right_finger"
-        origin_xyz="0 0 0.5"
+        origin_xyz="0 0 -0.01368"
         origin_rpy="0 -1.5708  0"
         scale = '0.001 0.001 0.001' />

Commit message: Aligned and working

File: src/xarm_ros/xarm_description/urdf/gripper/lite_gripper.urdf.xacro (robot description, xacro)
@@ -73,9 +73,10 @@
         material_name="${prefix}White"
         scale = '0.001 0.001 0.001' />
-      <xacro:common_link_collision
-        mesh_filename="gripper/omx/collision/omx_gripper_left_finger"
-        origin_xyz="0 0 0.0030"
-        origin_rpy="0 -1.5708 0"
-        scale = '0.001 0.001 0.001'/>
+        <collision>
+          <origin xyz="0 0 0.0030" rpy="0 -1.5708 0"/>
+          <geometry>
+            <box size="0.015 0.0200 0.058"/>
+          </geometry>
+        </collision>
     </link>
     <joint name="${prefix}left_finger_joint" type="prismatic">
@@ -103,9 +104,10 @@
         material_name="${prefix}White"
         scale = '0.001 0.001 0.001' />
-      <xacro:common_link_collision
-        mesh_filename="gripper/omx/collision/omx_gripper_right_finger"
-        origin_xyz="0 0 0.0030"
-        origin_rpy="0 -1.5708  0"
-        scale = '0.001 0.001 0.001' />
+        <collision>
+          <origin xyz="0 0 0.0030" rpy="0 -1.5708 0"/>
+          <geometry>
+            <box size="0.015 0.0200 0.058"/>
+          </geometry>
+        </collision>
     </link>
     <joint name="${prefix}right_finger_joint" type="prismatic">
